Commit message: feat: Add wall-mounting system to neurosurgical robot

File: urdf/robot_arm.urdf.xacro (robot description, xacro)
@@ -3,4 +3,11 @@
   <!-- Properties for easy modification -->
   <xacro:property name="PI" value="3.14159"/>
+  <!-- Wall mounting properties -->
+  <xacro:property name="wall_mount_height" value="0.15"/>
+  <xacro:property name="wall_mount_width" value="0.20"/>
+  <xacro:property name="wall_mount_depth" value="0.12"/>
+  <xacro:property name="wall_bracket_height" value="0.08"/>
+  <xacro:property name="wall_bracket_width" value="0.25"/>
+  <xacro:property name="wall_bracket_thickness" value="0.02"/>
   <!-- Realistic medical robot proportions -->
   <xacro:property name="base_height" value="0.08"/>
@@ -57,6 +64,142 @@
     <color rgba="1.0 0.8 0.0 1.0"/>
   </material>
-  <!-- World Link (operating room reference) -->
+  <!-- Wall mount material -->
+  <material name="wall_mount_steel">
+    <color rgba="0.7 0.7 0.75 1.0"/>
+  </material>
+  <!-- World Link (operating room wall reference) -->
   <link name="world"/>
+  <!-- Wall Bracket Link (Fixed to wall) -->
+  <link name="wall_bracket">
+    <!-- Main wall bracket plate -->
+    <visual>
+      <origin xyz="0 0 0" rpy="0 0 0"/>
+      <geometry>
+        <box size="${wall_bracket_width} ${wall_bracket_thickness} ${wall_bracket_height}"/>
+      </geometry>
+      <material name="wall_mount_steel"/>
+    </visual>
+    <!-- Reinforcement ribs -->
+    <visual>
+      <origin xyz="${wall_bracket_width/4} 0 0" rpy="0 0 0"/>
+      <geometry>
+        <box size="0.01 ${wall_bracket_thickness + 0.005} ${wall_bracket_height - 0.02}"/>
+      </geometry>
+      <material name="wall_mount_steel"/>
+    </visual>
+    <visual>
+      <origin xyz="${-wall_bracket_width/4} 0 0" rpy="0 0 0"/>
+      <geometry>
+        <box size="0.01 ${wall_bracket_thickness + 0.005} ${wall_bracket_height - 0.02}"/>
+      </geometry>
+      <material name="wall_mount_steel"/>
+    </visual>
+    <!-- Wall mounting bolts (decorative) -->
+    <visual>
+      <origin xyz="${wall_bracket_width/3} ${-wall_bracket_thickness/2 - 0.003} ${wall_bracket_height/3}" rpy="${PI/2} 0 0"/>
+      <geometry>
+        <cylinder radius="0.004" length="0.01"/>
+      </geometry>
+      <material name="cable_black"/>
+    </visual>
+    <visual>
+      <origin xyz="${-wall_bracket_width/3} ${-wall_bracket_thickness/2 - 0.003} ${wall_bracket_height/3}" rpy="${PI/2} 0 0"/>
+      <geometry>
+        <cylinder radius="0.004" length="0.01"/>
+      </geometry>
+      <material name="cable_black"/>
+    </visual>
+    <visual>
+      <origin xyz="${wall_bracket_width/3} ${-wall_bracket_thickness/2 - 0.003} ${-wall_bracket_height/3}" rpy="${PI/2} 0 0"/>
+      <geometry>
+        <cylinder radius="0.004" length="0.01"/>
+      </geometry>
+      <material name="cable_black"/>
+    </visual>
+    <visual>
+      <origin xyz="${-wall_bracket_width/3} ${-wall_bracket_thickness/2 - 0.003} ${-wall_bracket_height/3}" rpy="${PI/2} 0 0"/>
+      <geometry>
+        <cylinder radius="0.004" length="0.01"/>
+      </geometry>
+      <material name="cable_black"/>
+    </visual>
+    <collision>
+      <origin xyz="0 0 0" rpy="0 0 0"/>
+      <geometry>
+        <box size="${wall_bracket_width} ${wall_bracket_thickness} ${wall_bracket_height}"/>
+      </geometry>
+    </collision>
+    <inertial>
+      <mass value="2.8"/>
+      <origin xyz="0 0 0" rpy="0 0 0"/>
+      <inertia ixx="0.025" ixy="0" ixz="0" iyy="0.035" iyz="0" izz="0.045"/>
+    </inertial>
+  </link>
+  <!-- Wall Mount Housing Link (Extends from wall) -->
+  <link name="wall_mount">
+    <!-- Main mounting arm -->
+    <visual>
+      <origin xyz="0 ${wall_mount_depth/2} 0" rpy="${PI/2} 0 0"/>
+      <geometry>
+        <cylinder radius="0.025" length="${wall_mount_depth}"/>
+      </geometry>
+      <material name="wall_mount_steel"/>
+    </visual>
+    <!-- Mounting platform -->
+    <visual>
+      <origin xyz="0 ${wall_mount_depth} 0" rpy="0 0 0"/>
+      <geometry>
+        <box size="${wall_mount_width} ${wall_mount_height} 0.02"/>
+      </geometry>
+      <material name="wall_mount_steel"/>
+    </visual>
+    <!-- Platform reinforcement -->
+    <visual>
+      <origin xyz="0 ${wall_mount_depth + wall_mount_height/2} 0" rpy="0 0 0"/>
+      <geometry>
+        <box size="${wall_mount_width - 0.02} 0.01 0.025"/>
+      </geometry>
+      <material name="wall_mount_steel"/>
+    </visual>
+    <!-- Cable management channel -->
+    <visual>
+      <origin xyz="${wall_mount_width/3} ${wall_mount_depth/2} 0" rpy="${PI/2} 0 0"/>
+      <geometry>
+        <cylinder radius="0.008" length="${wall_mount_depth}"/>
+      </geometry>
+      <material name="cable_black"/>
+    </visual>
+    <!-- Safety markings -->
+    <visual>
+      <origin xyz="0 ${wall_mount_depth + wall_mount_height - 0.005} 0.011" rpy="0 0 0"/>
+      <geometry>
+        <box size="${wall_mount_width - 0.01} 0.01 0.002"/>
+      </geometry>
+      <material name="safety_orange"/>
+    </visual>
+    <collision>
+      <origin xyz="0 ${wall_mount_depth/2} 0" rpy="0 0 0"/>
+      <geometry>
+        <box size="${wall_mount_width} ${wall_mount_depth} ${wall_mount_height}"/>
+      </geometry>
+    </collision>
+    <inertial>
+      <mass value="4.2"/>
+      <origin xyz="0 ${wall_mount_depth/2} 0" rpy="0 0 0"/>
+      <inertia ixx="0.045" ixy="0" ixz="0" iyy="0.035" iyz="0" izz="0.065"/>
+    </inertial>
+  </link>
+  <!-- World to Wall Bracket Joint (fixed to wall) -->
+  <joint name="world_to_wall_bracket" type="fixed">
+    <parent link="world"/>
+    <child link="wall_bracket"/>
+    <origin xyz="0 0 0" rpy="0 0 0"/>
+  </joint>
+  <!-- Wall Bracket to Mount Joint (fixed extension from wall) -->
+  <joint name="wall_bracket_to_mount" type="fixed">
+    <parent link="wall_bracket"/>
+    <child link="wall_mount"/>
+    <origin xyz="0 ${wall_bracket_thickness/2} 0" rpy="0 0 0"/>
+  </joint>
   <!-- Base Link Assembly (Professional base with motor housing) -->
   <link name="base_link">
@@ -118,9 +261,9 @@
     </inertial>
   </link>
-  <!-- World to Base Joint (fixed mounting) -->
-  <joint name="world_to_base" type="fixed">
-    <parent link="world"/>
+  <!-- Wall Mount to Base Joint (robot mounts on wall platform) -->
+  <joint name="wall_mount_to_base" type="fixed">
+    <parent link="wall_mount"/>
     <child link="base_link"/>
-    <origin xyz="0 0 0" rpy="0 0 0"/>
+    <origin xyz="0 ${wall_mount_depth + wall_mount_height} 0" rpy="0 0 0"/>
   </joint>
   <!-- Shoulder Link Assembly -->

Commit message: Update with scene objects, constraints and coordinates inputs

File: urdf/robot_arm.urdf.xacro (robot description, xacro)
@@ -3,4 +3,8 @@
   <!-- Properties for easy modification -->
   <xacro:property name="PI" value="3.14159"/>
+  <!-- Wall plate properties -->
+  <xacro:property name="plate_width" value="0.8"/>
+  <xacro:property name="plate_height" value="0.6"/>
+  <xacro:property name="plate_thickness" value="0.05"/>
   <!-- Wall mounting properties -->
   <xacro:property name="wall_mount_height" value="0.15"/>
@@ -68,6 +72,64 @@
     <color rgba="0.7 0.7 0.75 1.0"/>
   </material>
-  <!-- World Link (operating room wall reference) -->
-  <link name="world"/>
+  <!-- Wall plate material -->
+  <material name="wall_surface">
+    <color rgba="0.9 0.9 0.92 1.0"/>
+  </material>
+  <material name="mounting_holes">
+    <color rgba="0.3 0.3 0.3 1.0"/>
+  </material>
+  <!-- World Link (FIXED - Wall bottom now sits at grid level) -->
+  <link name="world">
+    <!-- Main wall plate surface - MOVED UP so bottom sits at Z=0 -->
+    <visual>
+      <origin xyz="0 0 ${plate_height/2}" rpy="0 0 0"/>
+      <geometry>
+        <box size="${plate_width} ${plate_thickness} ${plate_height}"/>
+      </geometry>
+      <material name="wall_surface"/>
+    </visual>
+    <!-- Mounting holes (decorative) - ADJUSTED for new wall position -->
+    <visual>
+      <origin xyz="0.2 ${-plate_thickness/2 - 0.002} ${plate_height/2 + 0.15}" rpy="${PI/2} 0 0"/>
+      <geometry>
+        <cylinder radius="0.005" length="0.008"/>
+      </geometry>
+      <material name="mounting_holes"/>
+    </visual>
+    <visual>
+      <origin xyz="-0.2 ${-plate_thickness/2 - 0.002} ${plate_height/2 + 0.15}" rpy="${PI/2} 0 0"/>
+      <geometry>
+        <cylinder radius="0.005" length="0.008"/>
+      </geometry>
+      <material name="mounting_holes"/>
+    </visual>
+    <visual>
+      <origin xyz="0.2 ${-plate_thickness/2 - 0.002} ${plate_height/2 - 0.15}" rpy="${PI/2} 0 0"/>
+      <geometry>
+        <cylinder radius="0.005" length="0.008"/>
+      </geometry>
+      <material name="mounting_holes"/>
+    </visual>
+    <visual>
+      <origin xyz="-0.2 ${-plate_thickness/2 - 0.002} ${plate_height/2 - 0.15}" rpy="${PI/2} 0 0"/>
+      <geometry>
+        <cylinder radius="0.005" length="0.008"/>
+      </geometry>
+      <material name="mounting_holes"/>
+    </visual>
+    <!-- Collision - MOVED UP to match visual -->
+    <collision>
+      <origin xyz="0 0 ${plate_height/2}" rpy="0 0 0"/>
+      <geometry>
+        <box size="${plate_width} ${plate_thickness} ${plate_height}"/>
+      </geometry>
+    </collision>
+    <!-- Inertial properties - MOVED UP to match -->
+    <inertial>
+      <mass value="5.0"/>
+      <origin xyz="0 0 ${plate_height/2}" rpy="0 0 0"/>
+      <inertia ixx="0.6" ixy="0" ixz="0" iyy="0.88" iyz="0" izz="0.53"/>
+    </inertial>
+  </link>
   <!-- Wall Bracket Link (Fixed to wall) -->
   <link name="wall_bracket">
@@ -190,9 +252,9 @@
     </inertial>
   </link>
-  <!-- World to Wall Bracket Joint (fixed to wall) -->
+  <!-- World to Wall Bracket Joint (fixed to wall plate) -->
   <joint name="world_to_wall_bracket" type="fixed">
     <parent link="world"/>
     <child link="wall_bracket"/>
-    <origin xyz="0 0 0" rpy="0 0 0"/>
+    <origin xyz="0 ${plate_thickness/2} ${plate_height/2}" rpy="0 0 0"/>
   </joint>
   <!-- Wall Bracket to Mount Joint (fixed extension from wall) -->
